File: kicad/Schwingkreis/Untitled/Untitled.kicad_sch (KiCad schematic)
At the start: 0 parts

Commit message: .
Parts:
- added C1, C2: C, symbol Device:C
- added L1, L2: L, symbol Device:L
- added Q1, Q2: NMOS, symbol Simulation_SPICE:NMOS
- added R1, R2: R, symbol Device:R
- added V1: 1, symbol Simulation_SPICE:VDC
Connections:
- new net: C1.1, C2.1, L1.1, L2.1, R1.1, R2.1, V1.1
- new net: C2.2, L2.2, Q1.2 (G), Q2.1 (D), R2.2
- new net: C1.2, L1.2, Q1.1 (D), Q2.2 (G), R1.2
- new net 0: Q1.3 (S), Q2.3 (S), V1.2
