File: Testprojekt/Testprojekt.kicad_pcb (KiCad board)
At the start: 2 copper layers, 7 parts, among them Q1 NMOS

Commit message: Testprojekt Update
Connections:
- Q1 pad 3: Net-(Q1-S) -> GND
- TP1 pad 1: Net-(R3-Pad1) -> /VG
Changed lines of the file:
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@@
 			(layers "F.Cu" "F.Mask" "F.Paste")
 			(roundrect_rratio 0.25)
-			(net "Net-(Q1-S)")
+			(net "GND")
 			(pinfunction "S_3")
 			(pintype "passive")
@@
 			(layers "*.Cu" "*.Mask")
 			(remove_unused_layers no)
-			(net "Net-(R3-Pad1)")
+			(net "/VG")
 			(pinfunction "1_1")
 			(pintype "passive")
