File: Testprojekt/Testprojekt.kicad_sch (KiCad schematic)
At the start: 9 parts, among them Q1 NMOS

Commit message: Testprojekt Update
Parts:
- removed R2: 39K, Resistor_SMD:R_0603_1608Metric, symbol Device:R
- removed R3: 600R, Resistor_SMD:R_0603_1608Metric, symbol Device:R
- added TP4: TestPoint, TestPoint:TestPoint_Loop_D2.60mm_Drill0.9mm_Beaded, symbol Connector:TestPoint
- R1: value 75K -> 1K
Connections:
- net GND: now also Q1.3 (S)
- net VG: now also TP1.1, V1.1
- net vd: now also TP4.1
Changed lines of the file:
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@@
 	(paper "A4")
+	(junction
+		(at 148.59 99.06)
+		(diameter 0)
+		(color 0 0 0 0)
+	)
 	(junction
 		(at 163.83 123.19)
@@
 	(wire
 		(pts
+			(xy 157.48 99.06) (xy 148.59 99.06)
+		)
+		(stroke
+			(width 0)
+			(type default)
+		)
+	)
+	(wire
+		(pts
 			(xy 163.83 107.95) (xy 163.83 123.19)
 		)
@@
 	(wire
 		(pts
-			(xy 138.43 105.41) (xy 140.97 105.41)
-		)
-		(stroke
-			(width 0)
-			(type default)
-		)
-	)
-	(wire
-		(pts
-			(xy 148.59 110.49) (xy 148.59 113.03)
+			(xy 148.59 110.49) (xy 148.59 123.19)
 		)
 		(stroke
@@
 	(wire
 		(pts
-			(xy 148.59 97.79) (xy 148.59 100.33)
-		)
-		(stroke
-			(width 0)
-			(type default)
-		)
-	)
-	(wire
-		(pts
-			(xy 128.27 105.41) (xy 130.81 105.41)
+			(xy 148.59 97.79) (xy 148.59 99.06)
+		)
+		(stroke
+			(width 0)
+			(type default)
+		)
+	)
+	(wire
+		(pts
+			(xy 148.59 99.06) (xy 148.59 100.33)
+		)
+		(stroke
+			(width 0)
+			(type default)
+		)
+	)
+	(wire
+		(pts
+			(xy 128.27 105.41) (xy 140.97 105.41)
+		)
+		(stroke
+			(width 0)
+			(type default)
+		)
+	)
+	(wire
+		(pts
+			(xy 157.48 93.98) (xy 157.48 99.06)
 		)
 		(stroke
@@
 	(wire
 		(pts
-			(xy 148.59 120.65) (xy 148.59 123.19)
-		)
-		(stroke
-			(width 0)
-			(type default)
-		)
-	)
-	(wire
-		(pts
 			(xy 128.27 109.22) (xy 128.27 105.41)
+		)
+		(stroke
+			(width 0)
+			(type default)
+		)
+	)
+	(wire
+		(pts
+			(xy 167.64 93.98) (xy 157.48 93.98)
 		)
 		(stroke
@@
 			)
 		)
-		(property "Value" "75K"
+		(property "Value" "1K"
 			(at 151.13 95.2499 0)
 			(show_name no)
@@
 	)
 	(symbol
-		(lib_id "Device:R")
-		(at 148.59 116.84 0)
+		(lib_id "Connector:TestPoint")
+		(at 167.64 93.98 270)
 		(unit 1)
 		(body_style 1)
-		(exclude_from_sim no)
+		(exclude_from_sim yes)
 		(in_bom yes)
 		(on_board yes)
@@
 		(dnp no)
 		(fields_autoplaced yes)
-		(property "Reference" "R2"
-			(at 151.13 115.5699 0)
-			(show_name no)
-			(do_not_autoplace no)
-			(effects
-				(font
-					(size 1.27 1.27)
-				)
-				(justify left)
-			)
-		)
-		(property "Value" "39K"
-			(at 151.13 118.1099 0)
-			(show_name no)
-			(do_not_autoplace no)
-			(effects
-				(font
-					(size 1.27 1.27)
-				)
-				(justify left)
-			)
-		)
-		(property "Footprint" "Resistor_SMD:R_0603_1608Metric"
-			(at 146.812 116.84 90)
+		(property "Reference" "TP4"
+			(at 172.72 92.7099 90)
+			(show_name no)
+			(do_not_autoplace no)
+			(effects
+				(font
+					(size 1.27 1.27)
+				)
+				(justify left)
+			)
+		)
+		(property "Value" "TestPoint"
+			(at 172.72 95.2499 90)
+			(show_name no)
+			(do_not_autoplace no)
+			(effects
+				(font
+					(size 1.27 1.27)
+				)
+				(justify left)
+			)
+		)
+		(property "Footprint" "TestPoint:TestPoint_Loop_D2.60mm_Drill0.9mm_Beaded"
+			(at 167.64 99.06 0)
 			(hide yes)
 			(show_name no)
@@
 		)
 		(property "Datasheet" ""
-			(at 148.59 116.84 0)
-			(hide yes)
-			(show_name no)
-			(do_not_autoplace no)
-			(effects
-				(font
-					(size 1.27 1.27)
-				)
-			)
-		)
-		(property "Description" "Resistor"
-			(at 148.59 116.84 0)
+			(at 167.64 99.06 0)
+			(hide yes)
+			(show_name no)
+			(do_not_autoplace no)
+			(effects
+				(font
+					(size 1.27 1.27)
+				)
+			)
+		)
+		(property "Description" "test point"
+			(at 167.64 93.98 0)
 			(hide yes)
 			(show_name no)
@@
 		)
 		(pin "1"
-		)
-		(pin "2"
 		)
 		(instances
 			(project "Testprojekt"
 				(path "/faea5e50-0203-44c8-a22d-e350243817e9"
-					(reference "R2")
+					(reference "TP4")
 					(unit 1)
 				)
@@
 			)
 		)
-		(property "Sim.Device" "NMOS"
+		(property "Sim.Device" "NPN"
 			(at 146.05 122.555 0)
 			(hide yes)
@@
 			)
 		)
-		(property "Sim.Type" "VDMOS"
+		(property "Sim.Type" "GUMMELPOON"
 			(at 146.05 124.46 0)
 			(hide yes)
@@
 			)
 		)
-		(property "Sim.Pins" "1=D 2=G 3=S"
+		(property "Sim.Pins" "1=C 2=B 3=E"
 			(at 146.05 120.65 0)
+			(hide yes)
+			(show_name no)
+			(do_not_autoplace no)
+			(effects
+				(font
+					(size 1.27 1.27)
+				)
+			)
+		)
+		(property "Sim.Library" "spicelibs\\elk.lib"
+			(at 146.05 105.41 0)
+			(hide yes)
+			(show_name no)
+			(do_not_autoplace no)
+			(effects
+				(font
+					(size 1.27 1.27)
+				)
+			)
+		)
+		(property "Sim.Name" "Q2N3904"
+			(at 146.05 105.41 0)
 			(hide yes)
 			(show_name no)
@@
 					(unit 1)
 				)
-			)
-		)
-	)
-	(symbol
-		(lib_id "Device:R")
-		(at 134.62 105.41 90)
-		(unit 1)
-		(body_style 1)
-		(exclude_from_sim no)
-		(in_bom yes)
-		(on_board yes)
-		(in_pos_files yes)
-		(dnp no)
-		(fields_autoplaced yes)
-		(property "Reference" "R3"
-			(at 134.62 99.06 90)
-			(show_name no)
-			(do_not_autoplace no)
-			(effects
-				(font
-					(size 1.27 1.27)
-				)
-			)
-		)
-		(property "Value" "600R"
-			(at 134.62 101.6 90)
-			(show_name no)
-			(do_not_autoplace no)
-			(effects
-				(font
-					(size 1.27 1.27)
-				)
-			)
-		)
-		(property "Footprint" "Resistor_SMD:R_0603_1608Metric"
-			(at 134.62 107.188 90)
-			(hide yes)
-			(show_name no)
-			(do_not_autoplace no)
-			(effects
-				(font
-					(size 1.27 1.27)
-				)
-			)
-		)
-		(property "Datasheet" ""
-			(at 134.62 105.41 0)
-			(hide yes)
-			(show_name no)
-			(do_not_autoplace no)
-			(effects
-				(font
-					(size 1.27 1.27)
-				)
-			)
-		)
-		(property "Description" "Resistor"
-			(at 134.62 105.41 0)
-			(hide yes)
-			(show_name no)
-			(do_not_autoplace no)
-			(effects
-				(font
-					(size 1.27 1.27)
-				)
-			)
-		)
-		(pin "2"
-		)
-		(pin "1"
-		)
-		(instances
-			(project "Testprojekt"
-				(path "/faea5e50-0203-44c8-a22d-e350243817e9"
-					(reference "R3")
-					(unit 1)
-				)

Commit message: Ordner Code für Python Auswertung hinzugefügt
Other:
- note added: ".control wrdata NMOS.txt I(XQ1:1) write NMOS.raw .endc"
Changed lines of the file:
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@@
 	(generator_version "10.0")
 	(paper "A4")
+	(text ".control\nwrdata NMOS.txt I(XQ1:1) \nwrite NMOS.raw \n.endc"
+		(exclude_from_sim no)
+		(at 133.35 90.424 0)
+		(effects
+			(font
+				(size 1.27 1.27)
+			)
+		)
+	)
 	(junction
 		(at 148.59 99.06)
@@
 			)
 		)
-		(property "Sim.Device" "NPN"
+		(property "Sim.Device" "SUBCKT"
 			(at 146.05 122.555 0)
 			(hide yes)
@@
 			)
 		)
-		(property "Sim.Type" "GUMMELPOON"
-			(at 146.05 124.46 0)
-			(hide yes)
-			(show_name no)
-			(do_not_autoplace no)
-			(effects
-				(font
-					(size 1.27 1.27)
-				)
-			)
-		)
-		(property "Sim.Pins" "1=C 2=B 3=E"
+		(property "Sim.Pins" "1=1 2=2 3=3"
 			(at 146.05 120.65 0)
 			(hide yes)
@@
 			)
 		)
-		(property "Sim.Name" "Q2N3904"
+		(property "Sim.Name" "BS170/PLP"
 			(at 146.05 105.41 0)
 			(hide yes)
