File: kicad/VCO-Schwingkreis/VCO-Schwingkreis/VCO-Schwingkreis.kicad_sch (KiCad schematic)
At the start: 8 parts, among them Q1 NMOS, Q2 NMOS

Commit message: Anfang der Dokumentation
Other:
- note added: ".control wrdata VCO-Schwingkreis.txt write VCO-Schwingkreis.raw .endc"
- note removed: ".control wrdata VCO-Schwingkreis.txt write NMOS.raw .endc"
Changed lines of the file:
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@@
 		)
 	)
-	(text ".control\nwrdata VCO-Schwingkreis.txt\nwrite NMOS.raw\n.endc"
+	(text ".control\nwrdata VCO-Schwingkreis.txt\nwrite VCO-Schwingkreis.raw\n.endc"
 		(exclude_from_sim no)
 		(at 145.542 39.37 0)
