File: kicad/Wien-VCO/Wien-VCO.kicad_sch (KiCad schematic)
At the start: 22 parts, among them J1 J113, U1 ${SIM.NAME}

Commit message: Update Ordnerstruktur
Parts:
- added R10: 10K, Resistor_THT:R_Axial_DIN0207_L6.3mm_D2.5mm_P7.62mm_Horizontal, symbol Device:R
- added R11: 50K, Resistor_THT:R_Axial_DIN0207_L6.3mm_D2.5mm_P7.62mm_Horizontal, symbol Device:R
- added R12: 75K, Resistor_THT:R_Axial_DIN0207_L6.3mm_D2.5mm_P7.62mm_Horizontal, symbol Device:R
- added U2: ${SIM.NAME}, Library:TL082, symbol Simulation_SPICE:OPAMP
- C1, C2: footprint (none) -> Capacitor_THT:C_Rect_L10.0mm_W3.0mm_P7.50mm_MKS4
- C3: value 1nF -> 2nF; footprint (none) -> Capacitor_THT:C_Rect_L10.0mm_W3.0mm_P7.50mm_MKS4
- D1: value 1N4148 -> 1N6263
- D2, D3, D4, D5: value 1SV305 -> BB535/SIE; footprint (none) -> Diode_SMD:D_SOD-323F
- R1, R2, R4, R5, R6, R8, R9: footprint (none) -> Resistor_THT:R_Axial_DIN0207_L6.3mm_D2.5mm_P7.62mm_Horizontal
- R3: value 2K4 -> 2K22; footprint (none) -> Resistor_THT:R_Axial_DIN0207_L6.3mm_D2.5mm_P7.62mm_Horizontal
- R7: value 30R -> 1K; footprint (none) -> Resistor_THT:R_Axial_DIN0207_L6.3mm_D2.5mm_P7.62mm_Horizontal
- U1: footprint (none) -> Library:SOIC8-Adapter
- V3: value {Vstr} -> 0.5V
Connections:
- net 0: now also R12.2
- net VCC+: now also U2.3 (V+)
- net VCC-: now also R11.2, U2.4 (V-)
- net Vstr: now also R10.2, U2.1 (+), U2.5
- new net: R10.1, R11.1, R12.1, U2.2 (-)
Other:
- note added: "* Parameter .param R=1K .param C=17pF * Initial Condition .ic V(/Va)=1e-12 * Models .model 1N6263 D(Is=1.82u Rs=2.8 N=1.7 Cjo=2.65p M=0.333 tt=1.44n BV=60 Ibv=200n) .MODEL BB535/SIE D (IS=1.75E-15 N=1.043 RS=60E-3 XTI=3 EG=1.11 CJO=25.31E-12 M=1.064 VJ=3.022 FC=.5 BV=32 IBV=100E-9 TT=120E-9 ) * Output .control wrdata Wien-VCO.csv V(/Va) V(/Ve) write Wien-VCO.raw .endc"
- note removed: "* Parameter .param R=1K .param C=17p .param Vstr=2 * Initial Condition .ic V(/Va)=1e-12 * Options *.options reltol=0.005 trtol=4 method=gear *.options numdgt=7 .control wrdata Wien-VCO_MM.csv V(/Va) V(/Ve) write Wien-VCO_MM.raw .endc"
- company: (none) -> Mirco Ick / Torben Becker / Tassilo Hertling
- title: (none) -> Wie-Robinson-Brückenschwinger als VCO
- moved on the sheet: C1, C2, C3, D2, D3, D4, D5, J1, R1, R2, R3, R4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

Commit message: Layout erstellt
Parts:
- added C4, C5: 100nF, Capacitor_SMD:C_0603_1608Metric, symbol Device:C
- added H1, H2, H3, H4: MountingHole, MountingHole:MountingHole_3.2mm_M3, symbol Mechanical:MountingHole
- added TP1, TP2, TP3, TP4, TP5: TestPoint, TestPoint:TestPoint_Keystone_5010-5014_Multipurpose, symbol Connector:TestPoint
- R3: value 2K22 -> 2K23
- R8: value 10K -> 8K
Connections:
- net 0: now also C4.1, C5.1, TP3.1
- net VCC+: now also C4.2, TP4.1
- net VCC-: now also C5.2, TP5.1
- net Va: now also TP1.1
- net Vstr: now also TP2.1
Other:
- note added: "* Parameter .param R=3.275K .param C=2.7pF * Initial Condition .ic V(/Va)=1e-12 * Models .model 1N6263 D(Is=1.82u Rs=2.8 N=1.7 Cjo=2.65p M=0.333 tt=1.44n BV=60 Ibv=200n) .MODEL BB535/SIE D (IS=1.75E-15 N=1.043 RS=60E-3 XTI=3 EG=1.11 CJO=25.31E-12 M=1.064 VJ=3.022 FC=.5 BV=32 IBV=100E-9 TT=120E-9 ) * Output .control wrdata Wien-VCO.csv V(/Va) V(/Ve) write Wien-VCO.raw .endc"
- note removed: "* Parameter .param R=1K .param C=17pF * Initial Condition .ic V(/Va)=1e-12 * Models .model 1N6263 D(Is=1.82u Rs=2.8 N=1.7 Cjo=2.65p M=0.333 tt=1.44n BV=60 Ibv=200n) .MODEL BB535/SIE D (IS=1.75E-15 N=1.043 RS=60E-3 XTI=3 EG=1.11 CJO=25.31E-12 M=1.064 VJ=3.022 FC=.5 BV=32 IBV=100E-9 TT=120E-9 ) * Output .control wrdata Wien-VCO.csv V(/Va) V(/Ve) write Wien-VCO.raw .endc"
- moved on the sheet: V1, V3

Commit message: Layout angepasst
Parts:
- H1, H2, H3, H4: footprint MountingHole:MountingHole_3.2mm_M3 -> MountingHole:MountingHole_3.2mm_M3_ISO7380
Changed lines of the file:
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@@
 			)
 		)
-		(property "Footprint" "MountingHole:MountingHole_3.2mm_M3"
+		(property "Footprint" "MountingHole:MountingHole_3.2mm_M3_ISO7380"
 			(at 265.43 146.05 0)
 			(hide yes)
@@
 			)
 		)
-		(property "Footprint" "MountingHole:MountingHole_3.2mm_M3"
+		(property "Footprint" "MountingHole:MountingHole_3.2mm_M3_ISO7380"
 			(at 265.43 156.21 0)
 			(hide yes)
@@
 			)
 		)
-		(property "Footprint" "MountingHole:MountingHole_3.2mm_M3"
+		(property "Footprint" "MountingHole:MountingHole_3.2mm_M3_ISO7380"
 			(at 265.43 151.13 0)
 			(hide yes)
@@
 			)
 		)
-		(property "Footprint" "MountingHole:MountingHole_3.2mm_M3"
+		(property "Footprint" "MountingHole:MountingHole_3.2mm_M3_ISO7380"
 			(at 265.43 161.29 0)
 			(hide yes)

Commit message: Layout finalisiert
Parts:
- removed U1: ${SIM.NAME}, Library:SOIC8-Adapter, symbol Simulation_SPICE:OPAMP
- added RV1: R_Potentiometer, Potentiometer_THT:Potentiometer_Bourns_3296Y_Vertical, symbol Device:R_Potentiometer
- added U3: MAX4104ESA_, MAX4104ESA_:SOIC127P600X175-8N, symbol MAX4104ESA_:MAX4104ESA_
- C3: value 2nF -> 1nF
- V3: value 0.5V -> 0V
Connections:
- net VCC+: now also U3.7 (VCC)
- net VCC-: now also U3.4 (VEE)
- net Va: now also RV1.3, U3.6 (OUT)
- net at C1.1, D5.2 (A), R1.2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: now also U3.3 (IN+)
- net Ve: no longer names the net of R3.1, R4.1, R8.1
- net Ve: now also RV1.2, U3.2 (IN-)
- new net: U3.1 (NC), U3.5 (NC), U3.8 (NC)
Other:
- note added: "* Parameter .param R=3.275K .param C=2.7pF * Initial Condition .ic V(/Va)=0.1 * Models .model 1N6263 D(Is=1.82u Rs=2.8 N=1.7 Cjo=2.65p M=0.333 tt=1.44n BV=60 Ibv=200n) .MODEL BB535/SIE D (IS=1.75E-15 N=1.043 RS=60E-3 XTI=3 EG=1.11 CJO=25.31E-12 M=1.064 VJ=3.022 FC=.5 BV=32 IBV=100E-9 TT=120E-9 ) * Output .control wrdata Wien-VCO.csv V(/Va) V(/Ve) write Wien-VCO.raw .endc"
- note removed: "* Parameter .param R=3.275K .param C=2.7pF * Initial Condition .ic V(/Va)=1e-12 * Models .model 1N6263 D(Is=1.82u Rs=2.8 N=1.7 Cjo=2.65p M=0.333 tt=1.44n BV=60 Ibv=200n) .MODEL BB535/SIE D (IS=1.75E-15 N=1.043 RS=60E-3 XTI=3 EG=1.11 CJO=25.31E-12 M=1.064 VJ=3.022 FC=.5 BV=32 IBV=100E-9 TT=120E-9 ) * Output .control wrdata Wien-VCO.csv V(/Va) V(/Ve) write Wien-VCO.raw .endc"
- moved on the sheet: C3, C4, C5, D1, R5, R7, TP1, TP3, TP4, TP5, V1, V2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
