File: kicad/Wien-Brücken-VCO_5MHz5/Wien-VCO.kicad_sch (KiCad schematic)
At the start: 15 parts, among them J1 J113, U1 LT1220

Commit message: 5.5 MHz Update
Parts:
- removed R6: 10K, symbol Device:R
- removed U1: LT1220, symbol Amplifier_Operational:TL081
- added R8: 10K, symbol Device:R
- added U1: ${SIM.NAME}, symbol Simulation_SPICE:OPAMP
- C3: value 10nF -> 1nF
- R3: value 2K -> 2K2
- R4: value 1K4 -> 1K2
- R5: value 10M -> 20K
- R7: value 470R -> 50R
Connections:
- net 0: now also J1.3 (S)
- net VCC+: now also U1.3 (V+)
- net VCC-: now also U1.4 (V-)
- net Va: now also U1.5
- net Ve: now also R3.1, R4.1, R8.1, U1.2 (-); no longer C1.1, R1.2, R2.1
- new net: C1.1, R1.2, R2.1, U1.1 (+)
- new net: J1.1 (D), R8.2
Other:
- note added: ".param R=1K .param C=25pF .model __D1 D(Vfwd=0.6 Cjo=0) .ic V(Net-_C2-Pad2_)=.001 .options reltol=0.005 trtol=4 method=gear .options numdgt=7"
- note removed: ".param R=100R .param C=280pF .model __D1 D(Vfwd=0.6) .ic V(Net-_C2-Pad2_)=.001"
